Commit message: changes 14

File: src/hyperdog-ros2/robots/descriptions/hyperdog_description/xacro/hyperdog_urdf_joints.xacro (robot description, xacro)
@@ -19,5 +19,5 @@
     <!-- *********  FR_hip joint ********* -->
     <joint name="FR_hip_joint" type="revolute">
-        <axis xyz="-1 0 0"/>
+        <axis xyz="1 0 0"/>
         <origin xyz="0.175 -0.066 0" rpy="0 0 0"/>
         <parent link="base_link"/>
@@ -41,5 +41,5 @@
     <!-- *********  BR_hip  ********* -->
     <joint name="BR_hip_joint" type="revolute">
-        <axis xyz="-1 0 0"/>
+        <axis xyz="1 0 0"/>
         <origin xyz="-0.175 -0.066 0" rpy="0 0 0"/>
         <parent link="base_link"/>
@@ -63,5 +63,5 @@
     <!-- *********  FR_uleg joint ********* -->
     <joint name="FR_uleg_joint" type="revolute">
-        <axis xyz="0 -1 0"/>
+        <axis xyz="0 1 0"/>
         <origin xyz="0 -0.104 0" rpy="0 0 0"/>
         <parent link="FR_hip_link"/>
@@ -74,5 +74,5 @@
     <!-- *********  FL_uleg  ********* -->
     <joint name="FL_uleg_joint" type="revolute">
-        <axis xyz="0 -1 0"/>
+        <axis xyz="0 1 0"/>
         <origin xyz="0 0.104 0" rpy="0 0 0"/>
         <parent link="FL_hip_link"/>
@@ -85,5 +85,5 @@
     <!-- *********  BR_uleg  ********* -->
     <joint name="BR_uleg_joint" type="revolute">
-        <axis xyz="0 -1 0"/>
+        <axis xyz="0 1 0"/>
         <origin xyz="0 -0.104 0" rpy="0 0 0"/>
         <parent link="BR_hip_link"/>
@@ -96,5 +96,5 @@
     <!-- *********  BL_uleg  ********* -->
     <joint name="BL_uleg_joint" type="revolute">
-        <axis xyz="0 -1 0"/>
+        <axis xyz="0 1 0"/>
         <origin xyz="0 0.104 0" rpy="0 0 0"/>
         <parent link="BL_hip_link"/>

Commit message: changes axis direction

File: src/hyperdog-ros2/robots/descriptions/hyperdog_description/xacro/hyperdog_urdf_joints.xacro (robot description, xacro)
@@ -19,5 +19,5 @@
     <!-- *********  FR_hip joint ********* -->
     <joint name="FR_hip_joint" type="revolute">
-        <axis xyz="1 0 0"/>
+        <axis xyz="-1 0 0"/>
         <origin xyz="0.175 -0.066 0" rpy="0 0 0"/>
         <parent link="base_link"/>
@@ -41,5 +41,5 @@
     <!-- *********  BR_hip  ********* -->
     <joint name="BR_hip_joint" type="revolute">
-        <axis xyz="1 0 0"/>
+        <axis xyz="-1 0 0"/>
         <origin xyz="-0.175 -0.066 0" rpy="0 0 0"/>
         <parent link="base_link"/>
@@ -63,5 +63,5 @@
     <!-- *********  FR_uleg joint ********* -->
     <joint name="FR_uleg_joint" type="revolute">
-        <axis xyz="0 1 0"/>
+        <axis xyz="0 -1 0"/>
         <origin xyz="0 -0.104 0" rpy="0 0 0"/>
         <parent link="FR_hip_link"/>
@@ -74,5 +74,5 @@
     <!-- *********  FL_uleg  ********* -->
     <joint name="FL_uleg_joint" type="revolute">
-        <axis xyz="0 1 0"/>
+        <axis xyz="0 -1 0"/>
         <origin xyz="0 0.104 0" rpy="0 0 0"/>
         <parent link="FL_hip_link"/>
@@ -85,5 +85,5 @@
     <!-- *********  BR_uleg  ********* -->
     <joint name="BR_uleg_joint" type="revolute">
-        <axis xyz="0 1 0"/>
+        <axis xyz="0 -1 0"/>
         <origin xyz="0 -0.104 0" rpy="0 0 0"/>
         <parent link="BR_hip_link"/>
@@ -96,5 +96,5 @@
     <!-- *********  BL_uleg  ********* -->
     <joint name="BL_uleg_joint" type="revolute">
-        <axis xyz="0 1 0"/>
+        <axis xyz="0 -1 0"/>
         <origin xyz="0 0.104 0" rpy="0 0 0"/>
         <parent link="BL_hip_link"/>
