Commit message: changes 15.9

File: src/hyperdog-ros2/robots/descriptions/hyperdog_description/xacro/consts.xacro (robot description, xacro)
@@ -9,15 +9,15 @@
     <xacro:property name="lleg_up_limit"  value="2.618"/>
     <xacro:property name="velocity"       value="1"/>
-    <xacro:property name="effort"         value="10"/>
+    <xacro:property name="effort"         value="100"/>
     <!-- joint dynamics -->
     <xacro:property name="use_dynamics" value="true"/>
     <xacro:macro name="hip_joint_dynamics">
-        <dynamics damping="0.01" friction="10000"/>
+        <dynamics damping="0.01" friction="1.0"/>
     </xacro:macro>
     <xacro:macro name="uleg_joint_dynamics">
-        <dynamics damping="0.01" friction="10000"/>
+        <dynamics damping="0.01" friction="1.0"/>
     </xacro:macro>
     <xacro:macro name="lleg_joint_dynamics">
-        <dynamics damping="0.01" friction="10000"/>
+        <dynamics damping="0.01" friction="1.0"/>
     </xacro:macro>
     <!-- configure inertia -->

Commit message: changes16.2

File: src/hyperdog-ros2/robots/descriptions/hyperdog_description/xacro/consts.xacro (robot description, xacro)
@@ -9,15 +9,15 @@
     <xacro:property name="lleg_up_limit"  value="2.618"/>
     <xacro:property name="velocity"       value="1"/>
-    <xacro:property name="effort"         value="100"/>
+    <xacro:property name="effort"         value="10"/>
     <!-- joint dynamics -->
     <xacro:property name="use_dynamics" value="true"/>
     <xacro:macro name="hip_joint_dynamics">
-        <dynamics damping="0.01" friction="1.0"/>
+        <dynamics damping="0.01" friction="10000.0"/>
     </xacro:macro>
     <xacro:macro name="uleg_joint_dynamics">
-        <dynamics damping="0.01" friction="1.0"/>
+        <dynamics damping="0.01" friction="10000.0"/>
     </xacro:macro>
     <xacro:macro name="lleg_joint_dynamics">
-        <dynamics damping="0.01" friction="1.0"/>
+        <dynamics damping="0.01" friction="1000.0"/>
     </xacro:macro>
     <!-- configure inertia -->

Commit message: changes 16.3

File: src/hyperdog-ros2/robots/descriptions/hyperdog_description/xacro/consts.xacro (robot description, xacro)
@@ -8,16 +8,16 @@
     <xacro:property name="lleg_low_limit" value="-1.57"/>
     <xacro:property name="lleg_up_limit"  value="2.618"/>
-    <xacro:property name="velocity"       value="1"/>
-    <xacro:property name="effort"         value="10"/>
+    <xacro:property name="velocity"       value="2.0"/>
+    <xacro:property name="effort"         value="20"/>
     <!-- joint dynamics -->
     <xacro:property name="use_dynamics" value="true"/>
     <xacro:macro name="hip_joint_dynamics">
-        <dynamics damping="0.01" friction="10000.0"/>
+        <dynamics damping="0.01" friction="10000000000000000000000000000000.0"/>
     </xacro:macro>
     <xacro:macro name="uleg_joint_dynamics">
-        <dynamics damping="0.01" friction="10000.0"/>
+        <dynamics damping="0.01" friction="10000000000000000000000000000000.0"/>
     </xacro:macro>
     <xacro:macro name="lleg_joint_dynamics">
-        <dynamics damping="0.01" friction="1000.0"/>
+        <dynamics damping="0.01" friction="10000000000000000000000000000000.0"/>
     </xacro:macro>
     <!-- configure inertia -->

File: src/hyperdog-ros2/robots/descriptions/hyperdog_description/xacro/hyperdog_gazebo.xacro (robot description, xacro)
@@ -36,9 +36,9 @@
     </xacro:macro>
     <xacro:macro name="gz_foot">
-        <mu1>0.9</mu1>
-        <mu2>0.9</mu2>
+        <mu1>1.0</mu1>
+        <mu2>1.0</mu2>
         <fdir1>1 0 0</fdir1>
         <kp value="1000000.0" />
-        <kd value="1.0" />
+        <kd value="10.0" />
         <maxVel>0.0</maxVel>
         <maxContacts>1</maxContacts>

Commit message: changes 16.4

File: src/hyperdog-ros2/robots/descriptions/hyperdog_description/xacro/consts.xacro (robot description, xacro)
@@ -13,11 +13,11 @@
     <xacro:property name="use_dynamics" value="true"/>
     <xacro:macro name="hip_joint_dynamics">
-        <dynamics damping="0.01" friction="10000000000000000000000000000000.0"/>
+        <dynamics damping="0.0" friction="1000.0"/>
     </xacro:macro>
     <xacro:macro name="uleg_joint_dynamics">
-        <dynamics damping="0.01" friction="10000000000000000000000000000000.0"/>
+        <dynamics damping="0.0" friction="1000.0"/>
     </xacro:macro>
     <xacro:macro name="lleg_joint_dynamics">
-        <dynamics damping="0.01" friction="10000000000000000000000000000000.0"/>
+        <dynamics damping="0.0" friction="1000.0"/>
     </xacro:macro>
     <!-- configure inertia -->

File: src/hyperdog-ros2/robots/descriptions/hyperdog_description/xacro/hyperdog_gazebo.xacro (robot description, xacro)
@@ -3,6 +3,6 @@
     <xacro:include filename="physics.xacro" />
     <xacro:macro name="gz_hip">
-        <mu1>0.8</mu1>
-        <mu2>0.8</mu2>
+        <mu1>0.1</mu1>   <!--0.8-->
+        <mu2>0.1</mu2>
         <kp value="1000000.0"/>
         <kd value="1.0"/>
@@ -12,6 +12,6 @@
     </xacro:macro>
     <xacro:macro name="gz_uleg">
-        <mu1>0.8</mu1>
-        <mu2>0.8</mu2>
+        <mu1>0.1</mu1>
+        <mu2>0.1</mu2>
         <kp value="1000000.0"/>
         <kd value="1.0"/>
@@ -23,6 +23,6 @@
     </xacro:macro>
     <xacro:macro name="gz_lleg">
-        <mu1>0.8</mu1>
-        <mu2>0.8</mu2>
+        <mu1>0.1</mu1>
+        <mu2>0.1</mu2>
         <fdir1>1 0 0</fdir1>
         <kp>1000000.0</kp>
@@ -36,6 +36,6 @@
     </xacro:macro>
     <xacro:macro name="gz_foot">
-        <mu1>1.0</mu1>
-        <mu2>1.0</mu2>
+        <mu1>0.1</mu1>
+        <mu2>0.1</mu2>
         <fdir1>1 0 0</fdir1>
         <kp value="1000000.0" />
@@ -46,5 +46,5 @@
         <self_collide>1</self_collide>
         <minDepth>0.001</minDepth>
-        <restitution_coefficient>1</restitution_coefficient>
+        <restitution_coefficient>0</restitution_coefficient>
         <threshold>0</threshold>
         <material>Gazebo/DarkGrey</material>
@@ -52,8 +52,8 @@
     <!-- body -->
     <gazebo reference="base_link">
-        <mu1>0.05</mu1>
-        <mu2>0.05</mu2>
-        <!-- <kp>1000000.0</kp>
-        <kd>1.0</kd> -->
+        <mu1>0.1</mu1>
+        <mu2>0.1</mu2>
+        <kp>1000000.0</kp>
+        <kd>1.0</kd>
         <maxVel>0.01</maxVel>
         <material>Gazebo/DarkGrey  </material>

File: src/hyperdog-ros2/robots/descriptions/hyperdog_description/xacro/physics.xacro (robot description, xacro)
@@ -5,5 +5,5 @@
     <xacro:macro name="inertial_body">
         <inertial>
-            <origin xyz="-0.006 0.00633 0.00214" rpy="0 0 0"/> <!-- 0.006, -0.000233, 0.00214 -->
+            <origin xyz="0.006 0.00233 0.00214" rpy="0 0 0"/> <!-- 0.006, -0.000233, 0.00214 "y" -0.006 0.00633 0.00214 -->
             <mass value="${body_mass}" />
             <inertia  ixx="0.011396658109874464" ixy="0" ixz="0" iyy="0.05486450023370329" iyz="0" izz="0.06098759357764758" />
